Commit message: Changed joint names

File: src/urdf/px.urdf (robot description, URDF)
Before this commit: robot px_robot, 7 links, 6 joints
Joints:
- removed joint joint_1
- removed joint joint_2
- removed joint joint_3
- removed joint joint_4
- added joint elbow: type revolute, parent link2, child link3, origin xyz=0.0 0.1065 0 rpy=0.0 0.0 0.0, axis 0 0 1, limit lower=-2.32 upper=2.32 effort=10.0 velocity=1.57
- added joint shoulder: type revolute, parent link1, child link2, origin xyz=0.0 0.0 0.042 rpy=1.5707 0.0 0.0, axis 0 0 1, limit lower=-2.32 upper=2.32 effort=10.0 velocity=1.57
- added joint waist: type revolute, parent base_link, child link1, origin xyz=0.0 0.0 0.09 rpy=0.0 0.0 0.0, axis 0 0 1, limit lower=-2.32 upper=2.32 effort=10.0 velocity=1.57
- added joint wrist: type revolute, parent link3, child link4, origin xyz=0.0 0.1065 0 rpy=0.0 0.0 0.0, axis 0 0 1, limit lower=-2.32 upper=2.32 effort=10.0 velocity=1.57

File: src/urdf/px_collision.urdf (robot description, URDF)
Before this commit: robot px_robot, 7 links, 6 joints
Joints:
- removed joint joint_1
- removed joint joint_2
- removed joint joint_3
- removed joint joint_4
- added joint elbow: type revolute, parent link2, child link3, origin xyz=0.0 0.1065 0 rpy=0.0 0.0 0.0, axis 0 0 1, limit lower=-2.32 upper=2.32 effort=10.0 velocity=1.57
- added joint shoulder: type revolute, parent link1, child link2, origin xyz=0.0 0.0 0.042 rpy=1.5707 0.0 0.0, axis 0 0 1, limit lower=-2.32 upper=2.32 effort=10.0 velocity=1.57
- added joint waist: type revolute, parent base_link, child link1, origin xyz=0.0 0.0 0.09 rpy=0.0 0.0 0.0, axis 0 0 1, limit lower=-2.32 upper=2.32 effort=10.0 velocity=1.57
- added joint wrist: type revolute, parent link3, child link4, origin xyz=0.0 0.1065 0 rpy=0.0 0.0 0.0, axis 0 0 1, limit lower=-2.32 upper=2.32 effort=10.0 velocity=1.57

File: src/urdf/px_transmission.urdf (robot description, URDF)
Before this commit: robot px_robot, 7 links, 6 joints
Joints:
- removed joint joint_1
- removed joint joint_2
- removed joint joint_3
- removed joint joint_4
- added joint elbow: type revolute, parent link2, child link3, origin xyz=0.0 0.1065 0 rpy=0.0 0.0 0.0, axis 0 0 1, limit lower=-2.32 upper=2.32 effort=10.0 velocity=1.57
- added joint shoulder: type revolute, parent link1, child link2, origin xyz=0.0 0.0 0.042 rpy=1.5707 0.0 0.0, axis 0 0 1, limit lower=-2.32 upper=2.32 effort=10.0 velocity=1.57
- added joint waist: type revolute, parent base_link, child link1, origin xyz=0.0 0.0 0.09 rpy=0.0 0.0 0.0, axis 0 0 1, limit lower=-2.32 upper=2.32 effort=10.0 velocity=1.57
- added joint wrist: type revolute, parent link3, child link4, origin xyz=0.0 0.1065 0 rpy=0.0 0.0 0.0, axis 0 0 1, limit lower=-2.32 upper=2.32 effort=10.0 velocity=1.57
