Commit message: Renamed package

File: src/urdf/px_collision.urdf (robot description, URDF)
Before this commit: robot px_robot, 7 links, 6 joints
Links:
- link base_link: geometry collision mesh filename=package://robotics-ros-2-phantomx-forward_kinematics/src/me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 scale=1 1 1; visual mesh filename=package://robotics-ros-2-phantomx-forward_kinematics/src/me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 scale=1 1 1
- link link1: geometry collision mesh filename=package://robotics-ros-2-phantomx-forward_kinematics/src/me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 scale=1 1 1; visual mesh filename=package://robotics-ros-2-phantomx-forward_kinematics/src/me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 scale=1 1 1
- link link2: geometry collision mesh filename=package://robotics-ros-2-phantomx-forward_kinematics/src/me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 scale=1 1 1; visual mesh filename=package://robotics-ros-2-phantomx-forward_kinematics/src/me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 scale=1 1 1
- link link3: geometry collision mesh filename=package://robotics-ros-2-phantomx-forward_kinematics/src/me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 scale=1 1 1; visual mesh filename=package://robotics-ros-2-phantomx-forward_kinematics/src/me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 scale=1 1 1
- link link4: geometry collision mesh filename=package://robotics-ros-2-phantomx-forward_kinematics/src/me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 scale=1 1 1; visual mesh filename=package://robotics-ros-2-phantomx-forward_kinematics/src/me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 scale=1 1 1
